Commit message: Adds a sample mapfile like 226

File: catkin_ws/src/duckietown_description/urdf/test_map.urdf.xacro (robot description, xacro)
@@ -2,6 +2,10 @@
 <robot name="duckietown" xmlns:xacro="http://www.ros.org/wiki/xacro">
     <!-- Parameters -->
-    <xacro:property name="tile_width" value="0.6096" />
+    <xacro:property name="tile_width" value="0.595" />
     <xacro:property name="tile_thickness" value="0.01" />
+    <xacro:property name="pos_0" value="0.02 0" />
+    <xacro:property name="pos_1" value="0 0.02" />
+    <xacro:property name="pos_2" value="-0.02 0" />
+    <xacro:property name="pos_3" value="0 -0.02" />
     <!-- Include the tile and tag macros -->
     <xacro:include filename="$(find duckietown_description)/urdf/macros.urdf.xacro" />
@@ -9,9 +13,78 @@
     <link name="world" />
     <!-- Describe the tiles -->
-    <xacro:tile x="0" y="0" type="tile" rotation="0" />
-    <xacro:tile x="0" y="1" type="tile" rotation="0" />
-    <xacro:tile x="0" y="2" type="tile" rotation="0" />
-    <xacro:tile x="1" y="0" type="tile" rotation="90" />
-    <xacro:tile x="1" y="1" type="tile" rotation="0" />
-    <xacro:tile x="1" y="2" type="tile" rotation="270" />
+    <xacro:tile x="0" y="0" type="turn" rotation="270" />
+    <xacro:tile x="0" y="1" type="straight" rotation="90" />
+    <xacro:tile x="0" y="2" type="3way" rotation="270" />
+    <xacro:tile x="0" y="3" type="straight" rotation="90" />
+    <xacro:tile x="0" y="4" type="straight" rotation="90" />
+    <xacro:tile x="0" y="5" type="3way" rotation="270" />
+    <xacro:tile x="0" y="6" type="straight" rotation="90" />
+    <xacro:tile x="0" y="7" type="straight" rotation="90" />
+    <xacro:tile x="0" y="8" type="straight" rotation="90" />
+    <xacro:tile x="0" y="9" type="turn" rotation="180" />
+    <xacro:tile x="1" y="0" type="straight" rotation="0" />
+    <xacro:tile x="1" y="1" type="empty" rotation="0" />
+    <xacro:tile x="1" y="2" type="straight" rotation="0" />
+    <xacro:tile x="1" y="3" type="empty" rotation="0" />
+    <xacro:tile x="1" y="4" type="empty" rotation="0" />
+    <xacro:tile x="1" y="5" type="straight" rotation="0" />
+    <xacro:tile x="1" y="6" type="empty" rotation="0" />
+    <xacro:tile x="1" y="7" type="empty" rotation="0" />
+    <xacro:tile x="1" y="8" type="empty" rotation="0" />
+    <xacro:tile x="1" y="9" type="straight" rotation="0" />
+    <xacro:tile x="2" y="0" type="straight" rotation="0" />
+    <xacro:tile x="2" y="1" type="empty" rotation="0" />
+    <xacro:tile x="2" y="2" type="turn" rotation="0" />
+    <xacro:tile x="2" y="3" type="straight" rotation="90" />
+    <xacro:tile x="2" y="4" type="straight" rotation="90" />
+    <xacro:tile x="2" y="5" type="4way" rotation="0" />
+    <xacro:tile x="2" y="6" type="straight" rotation="90" />
+    <xacro:tile x="2" y="7" type="turn" rotation="180" />
+    <xacro:tile x="2" y="8" type="empty" rotation="0" />
+    <xacro:tile x="2" y="9" type="straight" rotation="0" />
+    <xacro:tile x="3" y="0" type="3way" rotation="0" />
+    <xacro:tile x="3" y="1" type="straight" rotation="90" />
+    <xacro:tile x="3" y="2" type="straight" rotation="90" />
+    <xacro:tile x="3" y="3" type="turn" rotation="180" />
+    <xacro:tile x="3" y="4" type="empty" rotation="0" />
+    <xacro:tile x="3" y="5" type="straight" rotation="0" />
+    <xacro:tile x="3" y="6" type="empty" rotation="0" />
+    <xacro:tile x="3" y="7" type="turn" rotation="0" />
+    <xacro:tile x="3" y="8" type="straight" rotation="90" />
+    <xacro:tile x="3" y="9" type="3way" rotation="180" />
+    <xacro:tile x="4" y="0" type="straight" rotation="0" />
+    <xacro:tile x="4" y="1" type="empty" rotation="0" />
+    <xacro:tile x="4" y="2" type="empty" rotation="0" />
+    <xacro:tile x="4" y="3" type="straight" rotation="0" />
+    <xacro:tile x="4" y="4" type="empty" rotation="0" />
+    <xacro:tile x="4" y="5" type="turn" rotation="0" />
+    <xacro:tile x="4" y="6" type="straight" rotation="90" />
+    <xacro:tile x="4" y="7" type="straight" rotation="90" />
+    <xacro:tile x="4" y="8" type="turn" rotation="180" />
+    <xacro:tile x="4" y="9" type="straight" rotation="0" />
+    <xacro:tile x="5" y="0" type="turn" rotation="0" />
+    <xacro:tile x="5" y="1" type="straight" rotation="90" />
+    <xacro:tile x="5" y="2" type="straight" rotation="90" />
+    <xacro:tile x="5" y="3" type="turn" rotation="90" />
+    <xacro:tile x="5" y="4" type="empty" rotation="0" />
+    <xacro:tile x="5" y="5" type="empty" rotation="0" />
+    <xacro:tile x="5" y="6" type="empty" rotation="0" />
+    <xacro:tile x="5" y="7" type="empty" rotation="0" />
+    <xacro:tile x="5" y="8" type="turn" rotation="0" />
+    <xacro:tile x="5" y="9" type="turn" rotation="90" />
+    <!-- Describe the tags -->
+    <xacro:tag id="100" x="0" y="3" pos="pos_3" rotation="270" />
+    <xacro:tag id="101" x="0" y="2" pos="pos_3" rotation="0" />
+    <xacro:tag id="102" x="1" y="2" pos="pos_3" rotation="90" />
+    <xacro:tag id="103" x="4" y="0" pos="pos_1" rotation="90" />
+    <xacro:tag id="104" x="3" y="0" pos="pos_0" rotation="0" />
+    <xacro:tag id="105" x="4" y="1" pos="pos_3" rotation="180" />
+    <xacro:tag id="106" x="0" y="6" pos="pos_3" rotation="270" />
+    <xacro:tag id="107" x="0" y="5" pos="pos_3" rotation="0" />
+    <xacro:tag id="108" x="1" y="5" pos="pos_3" rotation="90" />
+    <xacro:tag id="109" x="2" y="6" pos="pos_3" rotation="270" />
+    <xacro:tag id="110" x="2" y="5" pos="pos_3" rotation="0" />
+    <xacro:tag id="111" x="3" y="5" pos="pos_3" rotation="90" />
+    <xacro:tag id="112" x="3" y="6" pos="pos_3" rotation="180" />
+    <xacro:tag id="114" x="3" y="9" pos="pos_3" rotation="0" />
 </robot>
