Commit message: Adds xacro macros for tiles and tags to duckietown_description

File: catkin_ws/src/duckietown_description/urdf/macros.urdf.xacro (robot description, xacro)
@@ -2,14 +2,12 @@
 <robot name="macros" xmlns:xacro="http://www.ros.org/wiki/xacro">
     <xacro:property name="pi" value="3.14159265359" />
+    <!-- Defines a tile link and joint-->
     <xacro:macro name="tile" params="x y type rotation">
         <link name="tile_${x}_${y}">
             <visual>
-                <origin xyz="${tile_width/2} ${tile_width/2} ${-tile_thickness}" rpy="0 0 ${rotation * pi/180}"/>
+                <origin xyz="${tile_width/2} ${tile_width/2} ${-tile_thickness/2}" rpy="0 0 ${rotation * pi/180}"/>
                 <geometry>
-                    <box size="${tile_width} ${tile_width} ${tile_thickness}"/>
+                    <mesh filename="package://duckietown_description/urdf/meshes/${type}.dae" />
                 </geometry>
-                <material name="tile">
-                    <texture filename="package://duckietown_description/urdf/${type}.png" />
-                </material>
             </visual>
         </link>
@@ -20,3 +18,18 @@
         </joint>
     </xacro:macro>
+    <!-- Defines an april tag link and joint-->
+    <xacro:macro name="tag" params="id x y pos rotation">
+        <link name="tag_${id}">
+            <visual>
+                <geometry>
+                    <mesh filename="package://duckietown_description/urdf/meshes/sign_stop.dae" />
+                </geometry>
+            </visual>
+        </link>
+        <joint name="world_to_tag_${id}" type="fixed">
+            <parent link="tile_${x}_${y}" />
+            <child link="tag_${id}" />
+            <origin xyz="${pos_1} 0" rpy="0 0 ${rotation * pi/180}"/>
+        </joint>
+    </xacro:macro>
 </robot>

Commit message: Updates tiles

File: catkin_ws/src/duckietown_description/urdf/macros.urdf.xacro (robot description, xacro)
@@ -22,4 +22,5 @@
         <link name="tag_${id}">
             <visual>
+                <origin xyz="-0.0254 -0.0254 0" />
                 <geometry>
                     <mesh filename="package://duckietown_description/urdf/meshes/sign_stop.dae" />

Commit message: Adds invisible tiles at the border

File: catkin_ws/src/duckietown_description/urdf/macros.urdf.xacro (robot description, xacro)
@@ -2,13 +2,16 @@
 <robot name="macros" xmlns:xacro="http://www.ros.org/wiki/xacro">
     <xacro:property name="pi" value="3.14159265359" />
+    <xacro:property name="tile_thickness" value="0.01" />
     <!-- Defines a tile link and joint-->
-    <xacro:macro name="tile" params="x y type rotation">
+    <xacro:macro name="tile" params="x y type:=empty rotation:=0 visible:=true">
         <link name="tile_${x}_${y}">
-            <visual>
-                <origin xyz="${tile_width/2} ${tile_width/2} ${-tile_thickness/2}" rpy="0 0 ${rotation * pi/180}"/>
-                <geometry>
-                    <mesh filename="package://duckietown_description/urdf/meshes/${type}.dae" />
-                </geometry>
-            </visual>
+            <xacro:if value="${visible}" >
+                <visual>
+                    <origin xyz="${tile_width/2} ${tile_width/2} ${-tile_thickness/2}" rpy="0 0 ${rotation * pi/180}"/>
+                    <geometry>
+                        <mesh filename="package://duckietown_description/urdf/meshes/${type}.dae" />
+                    </geometry>
+                </visual>
+            </xacro:if>
         </link>
         <joint name="world_to_tile_${x}_${y}" type="fixed">
@@ -31,5 +34,5 @@
             <parent link="tile_${x}_${y}" />
             <child link="tag_${id}" />
-            <origin xyz="${pos_1} 0" rpy="0 0 ${rotation * pi/180}"/>
+            <origin xyz="${pos} 0" rpy="0 0 ${rotation * pi/180}"/>
         </joint>
     </xacro:macro>

File: catkin_ws/src/duckietown_description/urdf/test_map.urdf.xacro (robot description, xacro)
@@ -1,11 +1,11 @@
 <?xml version="1.0"?>
+<!-- WARNING: This file was auto-generated by <insert node name>. It should not be edited by hand. -->
 <robot name="duckietown" xmlns:xacro="http://www.ros.org/wiki/xacro">
     <!-- Parameters -->
     <xacro:property name="tile_width" value="0.595" />
-    <xacro:property name="tile_thickness" value="0.01" />
-    <xacro:property name="pos_0" value="0.02 0" />
-    <xacro:property name="pos_1" value="0 0.02" />
-    <xacro:property name="pos_2" value="-0.02 0" />
-    <xacro:property name="pos_3" value="0 -0.02" />
+    <xacro:property name="pos_0" value="0.04 0" />
+    <xacro:property name="pos_1" value="0 0.04" />
+    <xacro:property name="pos_2" value="-0.04 0" />
+    <xacro:property name="pos_3" value="0 -0.04" />
     <!-- Include the tile and tag macros -->
     <xacro:include filename="$(find duckietown_description)/urdf/macros.urdf.xacro" />
@@ -73,18 +73,38 @@
     <xacro:tile x="5" y="8" type="turn" rotation="0" />
     <xacro:tile x="5" y="9" type="turn" rotation="90" />
+    <!-- Empty border tiles -->
+    <xacro:tile x="6" y="0" visible="false" />
+    <xacro:tile x="6" y="1" visible="false" />
+    <xacro:tile x="6" y="2" visible="false" />
+    <xacro:tile x="6" y="3" visible="false" />
+    <xacro:tile x="6" y="4" visible="false" />
+    <xacro:tile x="6" y="5" visible="false" />
+    <xacro:tile x="6" y="6" visible="false" />
+    <xacro:tile x="6" y="7" visible="false" />
+    <xacro:tile x="6" y="8" visible="false" />
+    <xacro:tile x="6" y="9" visible="false" />
+    <xacro:tile x="6" y="10" visible="false" />
+    <xacro:tile x="5" y="10" visible="false" />
+    <xacro:tile x="4" y="10" visible="false" />
+    <xacro:tile x="3" y="10" visible="false" />
+    <xacro:tile x="2" y="10" visible="false" />
+    <xacro:tile x="1" y="10" visible="false" />
+    <xacro:tile x="0" y="10" visible="false" />
     <!-- Describe the tags -->
-    <xacro:tag id="100" x="0" y="3" pos="pos_3" rotation="270" />
-    <xacro:tag id="101" x="0" y="2" pos="pos_3" rotation="0" />
-    <xacro:tag id="102" x="1" y="2" pos="pos_3" rotation="90" />
-    <xacro:tag id="103" x="4" y="0" pos="pos_1" rotation="90" />
-    <xacro:tag id="104" x="3" y="0" pos="pos_0" rotation="0" />
-    <xacro:tag id="105" x="4" y="1" pos="pos_3" rotation="180" />
-    <xacro:tag id="106" x="0" y="6" pos="pos_3" rotation="270" />
-    <xacro:tag id="107" x="0" y="5" pos="pos_3" rotation="0" />
-    <xacro:tag id="108" x="1" y="5" pos="pos_3" rotation="90" />
-    <xacro:tag id="109" x="2" y="6" pos="pos_3" rotation="270" />
-    <xacro:tag id="110" x="2" y="5" pos="pos_3" rotation="0" />
-    <xacro:tag id="111" x="3" y="5" pos="pos_3" rotation="90" />
-    <xacro:tag id="112" x="3" y="6" pos="pos_3" rotation="180" />
-    <xacro:tag id="114" x="3" y="9" pos="pos_3" rotation="0" />
+    <xacro:tag id="100" x="0" y="3" pos="${pos_0}" rotation="270" />
+    <xacro:tag id="101" x="0" y="2" pos="${pos_0}" rotation="0" />
+    <xacro:tag id="102" x="1" y="2" pos="${pos_3}" rotation="90" />
+    <xacro:tag id="103" x="4" y="0" pos="${pos_1}" rotation="90" />
+    <xacro:tag id="104" x="3" y="0" pos="${pos_1}" rotation="0" />
+    <xacro:tag id="105" x="4" y="1" pos="${pos_3}" rotation="180" />
+    <xacro:tag id="106" x="0" y="6" pos="${pos_0}" rotation="270" />
+    <xacro:tag id="107" x="0" y="5" pos="${pos_0}" rotation="0" />
+    <xacro:tag id="108" x="1" y="5" pos="${pos_3}" rotation="90" />
+    <xacro:tag id="109" x="2" y="6" pos="${pos_3}" rotation="270" />
+    <xacro:tag id="110" x="2" y="5" pos="${pos_3}" rotation="0" />
+    <xacro:tag id="111" x="3" y="5" pos="${pos_3}" rotation="90" />
+    <xacro:tag id="112" x="3" y="6" pos="${pos_3}" rotation="180" />
+    <xacro:tag id="113" x="3" y="9" pos="${pos_3}" rotation="0" />
+    <xacro:tag id="114" x="3" y="10" pos="${pos_3}" rotation="270" />
+    <xacro:tag id="115" x="4" y="10" pos="${pos_3}" rotation="180" />
 </robot>
