Commit message: Fixes duckiebot visualization orientation bug

File: catkin_ws/src/duckietown_description/urdf/duckiebot.urdf.xacro (robot description, xacro)
@@ -1,7 +1,8 @@
 <?xml version="1.0"?>
 <robot name="duckiebot" xmlns:xacro="http://www.ros.org/wiki/xacro">
+    <xacro:property name="pi" value="3.14159265359" />
     <link name="duckiebot">
         <visual>
-            <origin xyz="0 0 0.04" />
+            <origin xyz="0 0 0.04" rpy="0 0 ${pi}"/>
             <geometry>
                 <mesh filename="package://duckietown_description/urdf/meshes/duckiebot.dae" />
