Commit message: added open house small ring map

File: catkin_ws/src/duckietown_description/urdf/open_house_dp6.urdf.xacro (robot description, xacro)
@@ -4,12 +4,12 @@
         <!--Parameters-->
         <xacro:property name="tile_width" value="0.595"/>
-        <xacro:property name="pos_0" value="0.125 0.035"/>
-        <xacro:property name="pos_1" value="0.035 0.125"/>
-        <xacro:property name="pos_2" value="-0.035 0.125"/>
-        <xacro:property name="pos_3" value="-0.125 0.035"/>
-        <xacro:property name="pos_4" value="-0.125 -0.035"/>
-        <xacro:property name="pos_5" value="-0.035 -0.125"/>
-        <xacro:property name="pos_6" value="0.035 -0.125"/>
-        <xacro:property name="pos_7" value="0.125 -0.035"/>
+        <xacro:property name="pos_0" value="0.09 0.035"/>
+        <xacro:property name="pos_1" value="0.035 0.09"/>
+        <xacro:property name="pos_2" value="-0.035 0.09"/>
+        <xacro:property name="pos_3" value="-0.09 0.035"/>
+        <xacro:property name="pos_4" value="-0.09 -0.035"/>
+        <xacro:property name="pos_5" value="-0.035 -0.09"/>
+        <xacro:property name="pos_6" value="0.035 -0.09"/>
+        <xacro:property name="pos_7" value="0.09 -0.035"/>
         <!--Include the tile and tag macros-->
         <xacro:include filename="$(find duckietown_description)/urdf/macros.urdf.xacro"/>
